Commit message: Align B2Z1 training and teleop low-level stack

File: gr00t/rl/third_party/visual_wholebody_lowlevel/resources/robots/b2z1/urdf/generated/b2z1_mount_0_x0p22_y0_z0p17.urdf (robot description, URDF)
Before this commit: robot b2_description, 29 links, 28 joints
Links:
- added link FL_calf_rotor, mass 0.2734
- added link FL_hip_rotor, mass 0.2734
- added link FL_thigh_rotor, mass 0.2734
- added link FR_calf_rotor, mass 0.2734
- added link FR_hip_rotor, mass 0.2734
- added link FR_thigh_rotor, mass 0.2734
- added link RL_calf_rotor, mass 0.2734
- added link RL_hip_rotor, mass 0.2734
- added link RL_thigh_rotor, mass 0.2734
- added link RR_calf_rotor, mass 0.2734
- added link RR_hip_rotor, mass 0.2734
- added link RR_thigh_rotor, mass 0.2734
- added link f_dc_link, mass 0.001
- added link f_oc_link, mass 0.001
- added link gripperMover, mass 0.27621302; collision mesh filename=../../meshes/z1_GripperMover.dae scale=1 1 1; visual mesh filename=../../meshes/z1_GripperMover.dae scale=1 1 1
- added link lidar_link, mass 0.001
- added link r_dc_link, mass 0.001
- added link r_oc_link, mass 0.001
- link FL_calf: geometry collision box size=0.342 0.04 0.047; visual mesh filename=../../meshes/FL_calf.dae
- link FL_foot: geometry collision sphere radius=0.032
- link FL_thigh: geometry collision box size=0.338 0.054 0.065; visual mesh filename=../../meshes/FL_thigh.dae
- link FR_calf: geometry collision box size=0.342 0.04 0.047; visual mesh filename=../../meshes/FR_calf.dae
- link FR_foot: geometry collision sphere radius=0.032
- link FR_hip: mass 2.256 -> 2.673
- link FR_thigh: geometry collision box size=0.338 0.054 0.065; visual mesh filename=../../meshes/FR_thigh.dae
- link RL_calf: geometry collision box size=0.342 0.04 0.047; visual mesh filename=../../meshes/RL_calf.dae
- link RL_foot: geometry collision sphere radius=0.032
- link RL_hip: mass 2.256 -> 2.673
- link RL_thigh: geometry collision box size=0.338 0.054 0.065; visual mesh filename=../../meshes/RL_thigh.dae
- link RR_calf: geometry collision box size=0.342 0.04 0.047; visual mesh filename=../../meshes/RR_calf.dae
- link RR_foot: geometry collision sphere radius=0.032
- link RR_thigh: geometry collision box size=0.338 0.054 0.065; visual mesh filename=../../meshes/RR_thigh.dae
- link base_link: geometry collision box size=0.568 0.295 0.255; visual mesh filename=../../meshes/base_link_no_lidar.dae
- link gripperStator: geometry collision mesh filename=../../meshes/z1_GripperStator.dae scale=1 1 1; visual mesh filename=../../meshes/z1_GripperStator.dae scale=1 1 1
- link gripper_link: mass 0.27621302 -> 0.001; geometry collision box size=0.01 0.01 0.01
- link imu_link: mass 4.19E-15 -> 0.001
- link link00: geometry collision cylinder length=0.03 radius=0.0325; visual mesh filename=../../meshes/z1_Link00.dae scale=1 1 1
- link link02: geometry collision cylinder length=0.051 radius=0.0325; collision cylinder length=0.102 radius=0.02
- link link04: geometry collision cylinder length=0.073 radius=0.0325; visual mesh filename=../../meshes/z1_Link04.dae scale=1 1 1
Joints:
- removed joint gripperStator
- added joint FL_calf_rotor_joint: type fixed, parent FL_thigh, child FL_calf_rotor, origin xyz=0 -0.05788 0 rpy=0 0 0
- added joint FL_hip_rotor_joint: type fixed, parent base_link, child FL_hip_rotor, origin xyz=0.20205 0.072 0 rpy=0 0 0
- added joint FL_thigh_rotor_joint: type fixed, parent FL_hip, child FL_thigh_rotor, origin xyz=0 -0.00798 0 rpy=0 0 0
- added joint FR_calf_rotor_joint: type fixed, parent FR_thigh, child FR_calf_rotor, origin xyz=0 0.05788 0 rpy=0 0 0
- added joint FR_hip_rotor_joint: type fixed, parent base_link, child FR_hip_rotor, origin xyz=0.20205 -0.072 0 rpy=0 0 0
- added joint FR_thigh_rotor_joint: type fixed, parent FR_hip, child FR_thigh_rotor, origin xyz=0 0.00798 0 rpy=0 0 0
- added joint RL_calf_rotor_joint: type fixed, parent RL_thigh, child RL_calf_rotor, origin xyz=0 -0.05788 0 rpy=0 0 0
- added joint RL_hip_rotor_joint: type fixed, parent base_link, child RL_hip_rotor, origin xyz=-0.20205 0.072 0 rpy=0 0 0
- added joint RL_thigh_rotor_joint: type fixed, parent RL_hip, child RL_thigh_rotor, origin xyz=0 -0.00798 0 rpy=0 0 0
- added joint RR_calf_rotor_joint: type fixed, parent RR_thigh, child RR_calf_rotor, origin xyz=0 0.05788 0 rpy=0 0 0
- added joint RR_hip_rotor_joint: type fixed, parent base_link, child RR_hip_rotor, origin xyz=-0.20205 -0.072 0 rpy=0 0 0
- added joint RR_thigh_rotor_joint: type fixed, parent RR_hip, child RR_thigh_rotor, origin xyz=0 0.00798 0 rpy=0 0 0
- added joint ee_gripper: type fixed, parent gripperStator, child gripper_link, origin xyz=0.135 0 0 rpy=0 0 0, axis 1 0 0
- added joint jointGripperStator: type fixed, parent link06, child gripperStator, origin xyz=0.051 0 0 rpy=-1.5707963267948966 0 0
- added joint joint_f_dc: type fixed, parent base_link, child f_dc_link, origin xyz=0.41251 0.024997 0.04765 rpy=-2.3562 0 -1.5708, axis 0 0 0
- added joint joint_f_oc: type fixed, parent base_link, child f_oc_link, origin xyz=0.39079 0 -0.013433 rpy=-1.5708 0 -1.5708, axis 0 0 0
- added joint joint_lidar: type fixed, parent base_link, child lidar_link, origin xyz=0.34218 0 0.17851 rpy=0 0 0, axis 0 0 0
- added joint joint_r_dc: type fixed, parent base_link, child r_dc_link, origin xyz=-0.4081 -0.025 0.024861 rpy=-2.3557 0 1.5708, axis 0 0 0
- added joint joint_r_oc: type fixed, parent base_link, child r_oc_link, origin xyz=-0.38451 0 -0.023249 rpy=-1.5708 0 1.5708, axis 0 0 0
- joint joint1: limit lower=-2.618 upper=2.618 effort=30.0 velocity=10 -> lower=-2.6179938779914944 upper=2.6179938779914944 effort=30.0 velocity=3.1415
- joint joint2: limit lower=0.0 upper=3.14 effort=60.0 velocity=10 -> lower=0.0 upper=2.9670597283903604 effort=60.0 velocity=3.1415
- joint joint3: limit lower=-4.78 upper=0.0 effort=30.0 velocity=10 -> lower=-2.8797932657906435 upper=0.0 effort=30.0 velocity=3.1415
- joint joint4: limit lower=-1.744 upper=1.57 effort=30.0 velocity=10 -> lower=-1.5184364492350666 upper=1.5184364492350666 effort=30.0 velocity=3.1415
- joint joint5: limit lower=-1.727 upper=1.727 effort=30.0 velocity=10 -> lower=-1.3439035240356338 upper=1.3439035240356338 effort=30.0 velocity=3.1415
- joint joint6: limit lower=-2.79 upper=2.79 effort=30.0 velocity=10 -> lower=-2.792526803190927 upper=2.792526803190927 effort=30.0 velocity=3.1415
- joint jointGripper: child gripper_link -> gripperMover; limit lower=-1.57 upper=0.0 effort=30.0 velocity=10 -> lower=-0.78539816339 upper=0.78539816339 effort=20.0 velocity=3.1415; origin xyz=0.049 0.0 0 rpy=0 0 0 -> xyz=0.049 0 0 rpy=0 0 0

Commit message: Align B2Z1 gripper collision hulls with lab30

File: gr00t/rl/third_party/visual_wholebody_lowlevel/resources/robots/b2z1/urdf/generated/b2z1_mount_0_x0p22_y0_z0p17.urdf (robot description, URDF)
Before this commit: robot b2_description, 47 links, 46 joints
Links:
- link base_link: geometry collision box size=0.206 0.12 0.10; collision box size=0.568 0.295 0.255
- link gripperMover: geometry collision mesh filename=../../meshes/gripper_collision_hulls/moving_000.obj scale=1 1 1; collision mesh filename=../../meshes/gripper_collision_hulls/moving_001.obj scale=1 1 1
- link gripperStator: geometry collision mesh filename=../../meshes/gripper_collision_hulls/fixed_000.obj scale=1 1 1; collision mesh filename=../../meshes/gripper_collision_hulls/fixed_001.obj scale=1 1 1
Joints:
- joint ee_gripper: origin xyz=0.135 0 0 rpy=0 0 0 -> xyz=0.049 0 0 rpy=0 0 0
- joint jointGripper: limit lower=-0.78539816339 upper=0.78539816339 effort=20.0 velocity=3.1415 -> lower=-1.0471975511965976 upper=0.0 effort=20.0 velocity=3.1415
